File: schematics/silentfan_with_relay.brd (EAGLE design)
At the start: 100 x 80 mm, 22 parts, among them T1 2N3904, T2 2N3904

Commit message: Add some POC schematics
Parts:
- removed PWR_GND, PWR_VCC12, PWR_VCC5: PIN1-2, con-faston:62221
- R4: value 50 -> 100
- moved R3 123.9 mm to (94.0, 50.8)
- moved LED1 116.9 mm to (88.9, 50.8)
- moved CTL_5V 116.8 mm to (91.4, 73.7)
- moved R2 115.0 mm to (83.8, 61.0), turned to 270 degrees
- moved R4 105.6 mm to (25.4, 61.0)
- moved CTL_ON_OFF_5V 101.9 mm to (91.4, 66.0)
- moved T2 95.1 mm to (58.4, 61.0)
- moved CTL_GND 94.4 mm to (91.4, 58.4)
- moved FO_GND 74.7 mm to (10.2, 17.8)
- moved FO_VCC 65.1 mm to (10.2, 25.4)
- moved FO_TACH 55.7 mm to (10.2, 33.0)
- moved FO_PWM 51.8 mm to (10.2, 40.6)
- moved R1 38.7 mm to (63.5, 63.5)
- moved T1 33.0 mm to (58.4, 66.0)
- moved U$1 20.3 mm to (49.5, 67.3), turned to 180 degrees
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Connections:
- removed net N$8: PWR_VCC5.1, R4.1
- net N$1: now also FI_VCC12.1, R4.1, U$1.COM-CLOSE; no longer FI_GND.1, FO_GND.1, PWR_GND.1
- net N$5: now also FI_GND.1, FO_GND.1; no longer PWR_VCC12.1, U$1.COM-CLOSE
Routing:
- net N$5: track 0.00 -> 60.3 mm
- net N$9: track 0.00 -> 59.0 mm
- net N$10: track 0.00 -> 57.4 mm
- net N$14: track 0.00 -> 40.1 mm
- net N$12: track 0.00 -> 34.7 mm
- net N$1: track 0.00 -> 34.4 mm
- net N$7: track 0.00 -> 31.5 mm
- net N$3: track 0.00 -> 29.9 mm
- net N$6: track 0.00 -> 11.8 mm
- net N$4: track 0.00 -> 10.2 mm
- net N$11: track 0.00 -> 9.67 mm
- net N$2: track 0.00 -> 5.71 mm
- net N$13: track 0.00 -> 2.67 mm
