File: schematics/silentfan_with_relay.sch (EAGLE design)
At the start: 22 parts, among them T1 2N3904, T2 2N3904

Commit message: Add some POC schematics
Parts:
- removed PWR_GND, PWR_VCC12, PWR_VCC5: PIN1-2, con-faston:PIN1-2
- R4: value 50 -> 100
Connections:
- removed net N$8: PWR_VCC5.1, R4.1
- net N$1: now also FI_VCC12.1, R4.1, U$1.COM-CLOSE; no longer FI_GND.1, FO_GND.1, PWR_GND.1
- net N$5: now also FI_GND.1, FO_GND.1; no longer PWR_VCC12.1, U$1.COM-CLOSE
Other:
- moved on the sheet: R4
Changed lines of the file:
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@@
 <part name="FO_TACH" library="con-faston" library_urn="urn:adsk.eagle:library:144" deviceset="PIN1-2" device="" package3d_urn="urn:adsk.eagle:package:6764/1"/>
 <part name="FO_PWM" library="con-faston" library_urn="urn:adsk.eagle:library:144" deviceset="PIN1-2" device="" package3d_urn="urn:adsk.eagle:package:6764/1"/>
-<part name="PWR_VCC12" library="con-faston" library_urn="urn:adsk.eagle:library:144" deviceset="PIN1-2" device="" package3d_urn="urn:adsk.eagle:package:6764/1"/>
-<part name="PWR_VCC5" library="con-faston" library_urn="urn:adsk.eagle:library:144" deviceset="PIN1-2" device="" package3d_urn="urn:adsk.eagle:package:6764/1"/>
-<part name="PWR_GND" library="con-faston" library_urn="urn:adsk.eagle:library:144" deviceset="PIN1-2" device="" package3d_urn="urn:adsk.eagle:package:6764/1"/>
 <part name="CTL_ON_OFF_5V" library="con-faston" library_urn="urn:adsk.eagle:library:144" deviceset="PIN1-2" device="" package3d_urn="urn:adsk.eagle:package:6764/1"/>
 <part name="CTL_GND" library="con-faston" library_urn="urn:adsk.eagle:library:144" deviceset="PIN1-2" device="" package3d_urn="urn:adsk.eagle:package:6764/1"/>
@@
 <part name="LED1" library="led" library_urn="urn:adsk.eagle:library:259" deviceset="LED" device="3MM" package3d_urn="urn:adsk.eagle:package:15797/1"/>
 <part name="R3" library="resistor" library_urn="urn:adsk.eagle:library:348" deviceset="R-EU_" device="0204/2V" package3d_urn="urn:adsk.eagle:package:25948/1" value="1k"/>
-<part name="R4" library="resistor" library_urn="urn:adsk.eagle:library:348" deviceset="R-EU_" device="0309/12" package3d_urn="urn:adsk.eagle:package:26089/1" value="50"/>
+<part name="R4" library="resistor" library_urn="urn:adsk.eagle:library:348" deviceset="R-EU_" device="0309/12" package3d_urn="urn:adsk.eagle:package:26089/1" value="100"/>
 </parts>
 <sheets>
@@
 <attribute name="NAME" x="96.52" y="77.47" size="1.778" layer="95" rot="MR180"/>
 </instance>
-<instance part="PWR_VCC12" gate="G$1" x="15.24" y="68.58" smashed="yes" rot="R180">
-<attribute name="NAME" x="10.16" y="69.85" size="1.778" layer="95" rot="R180"/>
-</instance>
-<instance part="PWR_VCC5" gate="G$1" x="15.24" y="66.04" smashed="yes" rot="R180">
-<attribute name="NAME" x="10.16" y="67.31" size="1.778" layer="95" rot="R180"/>
-</instance>
-<instance part="PWR_GND" gate="G$1" x="15.24" y="71.12" smashed="yes" rot="R180">
-<attribute name="NAME" x="10.16" y="72.39" size="1.778" layer="95" rot="R180"/>
-</instance>
 <instance part="CTL_ON_OFF_5V" gate="G$1" x="15.24" y="48.26" smashed="yes" rot="R180">
 <attribute name="NAME" x="10.16" y="49.53" size="1.778" layer="95" rot="R180"/>
@@
 <attribute name="VALUE" x="74.93" y="22.098" size="1.778" layer="96"/>
 </instance>
-<instance part="R4" gate="G$1" x="27.94" y="66.04" smashed="yes">
-<attribute name="NAME" x="29.21" y="62.4586" size="1.778" layer="95"/>
-<attribute name="VALUE" x="24.13" y="62.738" size="1.778" layer="96"/>
+<instance part="R4" gate="G$1" x="30.48" y="66.04" smashed="yes">
+<attribute name="NAME" x="31.75" y="62.4586" size="1.778" layer="95"/>
+<attribute name="VALUE" x="26.67" y="62.738" size="1.778" layer="96"/>
 </instance>
 </instances>
@@
 <net name="N$1" class="0">
 <segment>
-<pinref part="FI_GND" gate="G$1" pin="1"/>
-<pinref part="FO_GND" gate="G$1" pin="1"/>
-<wire x1="20.32" y1="83.82" x2="35.56" y2="83.82" width="0.1524" layer="91"/>
-<pinref part="PWR_GND" gate="G$1" pin="1"/>
-<wire x1="35.56" y1="83.82" x2="86.36" y2="83.82" width="0.1524" layer="91"/>
-<wire x1="20.32" y1="71.12" x2="35.56" y2="71.12" width="0.1524" layer="91"/>
-<wire x1="35.56" y1="71.12" x2="35.56" y2="83.82" width="0.1524" layer="91"/>
-<junction x="35.56" y="83.82"/>
+<pinref part="U$1" gate="G$1" pin="COM-CLOSE"/>
+<wire x1="45.72" y1="68.58" x2="91.44" y2="68.58" width="0.1524" layer="91"/>
+<wire x1="91.44" y1="68.58" x2="91.44" y2="45.72" width="0.1524" layer="91"/>
+<pinref part="FI_VCC12" gate="G$1" pin="1"/>
+<wire x1="45.72" y1="81.28" x2="45.72" y2="68.58" width="0.1524" layer="91"/>
+<wire x1="45.72" y1="81.28" x2="22.86" y2="81.28" width="0.1524" layer="91"/>
+<wire x1="22.86" y1="81.28" x2="20.32" y2="81.28" width="0.1524" layer="91"/>
+<wire x1="22.86" y1="81.28" x2="22.86" y2="66.04" width="0.1524" layer="91"/>
+<junction x="22.86" y="81.28"/>
+<pinref part="R4" gate="G$1" pin="1"/>
+<wire x1="22.86" y1="66.04" x2="25.4" y2="66.04" width="0.1524" layer="91"/>
 </segment>
 </net>
@@
 <pinref part="U$1" gate="G$1" pin="COM-OPEN"/>
 <wire x1="76.2" y1="66.04" x2="76.2" y2="45.72" width="0.1524" layer="91"/>
-<wire x1="33.02" y1="66.04" x2="76.2" y2="66.04" width="0.1524" layer="91"/>
+<wire x1="35.56" y1="66.04" x2="76.2" y2="66.04" width="0.1524" layer="91"/>
 <pinref part="R4" gate="G$1" pin="2"/>
-</segment>
-</net>
-<net name="N$5" class="0">
-<segment>
-<pinref part="PWR_VCC12" gate="G$1" pin="1"/>
-<wire x1="20.32" y1="68.58" x2="91.44" y2="68.58" width="0.1524" layer="91"/>
-<pinref part="U$1" gate="G$1" pin="COM-CLOSE"/>
-<wire x1="91.44" y1="68.58" x2="91.44" y2="45.72" width="0.1524" layer="91"/>
 </segment>
 </net>
@@
 </segment>
 </net>
-<net name="N$8" class="0">
-<segment>
-<pinref part="PWR_VCC5" gate="G$1" pin="1"/>
-<wire x1="20.32" y1="66.04" x2="22.86" y2="66.04" width="0.1524" layer="91"/>
-<pinref part="R4" gate="G$1" pin="1"/>
-</segment>
-</net>
+<net name="N$5" class="0">
+<segment>
+<pinref part="FO_GND" gate="G$1" pin="1"/>
+<pinref part="FI_GND" gate="G$1" pin="1"/>
+<wire x1="20.32" y1="83.82" x2="86.36" y2="83.82" width="0.1524" layer="91"/>
+</segment>
+</net>
